File: 02_Elements/MLP_ESPControlBoard_Rev_1/02_HW/MLP_ESPControlBoard_Rev_1.brd (EAGLE design)
At the start: 300 x 50 mm, 27 parts, among them Q1 T_UR0, Q2 T_UR0, U1 ESP-WROOM-03, X1 USB-MICROB

Commit message: Schematic Update
Advanced Schematic, not final
Parts:
- removed F_PW: PTCTHERMISTOR1206, SparkFun-PowerIC:PTC-1206
- removed J_MIDI: 22-05-7048-04, con-molex:7395-04
- removed J_PW: (no value), con-shiua-chyuan:SCD-014-A
- removed J_PZ_EXT: 22-05-7078-07, con-molex:7395-07
- removed R_LED_B, R_LED_G, R_LED_R: 330, adafruit:M1206
- removed R_MIDI_0, R_MIDI_1, R_MIDI_2: 220, adafruit:M1206
- removed U$1: CH340G, ch340g:SOIC16
- removed U_VR_5V: 7805T, adafruit:TO220H
- added C_DR_0, C_DR_1, C_ESP_2: 100uF, adafruit:C0805K
- added C_ESP_3: 470pF, adafruit:C0805K
- added C_VR_2: 330nF, adafruit:C1206K
- added C_VR_3: 100nF, adafruit:C1206K
- added D1, D2, D3: MBRA140, SparkFun-DiscreteSemi:SMA-DIODE
- added LED_PW1: (no value), adafruit:1206
- added MOTPOT_0, MOTPOT_1, MOTPOT_2: POLOLU_MOT_POT, PololuMotors:POLOLU_MOT_POT
- added R_ESP0, R_ESP1, R_ESP2, R_ESP3, R_ESP4: 12KOhm, adafruit:M0805
- added R_PW1: 330Ohm, adafruit:M1206
- added U_DR_0, U_DR_1: L293DD, st-microelectronics:SO20
- added U_UR0: CH340G, ch340g:SOIC16
- added U_VR_0: MC78GENERICDT, _hhn_78xx_79xx_NCV78xx_d2pak_dpak:DPAK-3
- added U_VR_1: UA78M33DCY, linear:SOT223
- added X_UR0: 12MHz, adafruit:CTS406
- C_UR0, C_UR1: device adafruit:C1812K -> adafruit:C0805K
- C_VR_0: value 18127C103KAT2A -> 330nF; device adafruit:C1812K -> adafruit:C1206K
- C_VR_1: value C1812F104K2RACTU -> 100nF; device adafruit:C1812K -> adafruit:C1206K
- LED_RGB: value RGBLED5050 -> (none); device adafruit:RGBLED5050 -> SparkFun-LED:WS2812B
- moved C_VR_0 467.5 mm to (-192.0, -115.0), turned to 0 degrees
- moved C_VR_1 466.2 mm to (-192.0, -119.0), turned to 0 degrees
- moved LED_RGB 341.1 mm to (-86.0, 16.0)
- moved LED_PW 302.0 mm to (-39.0, -36.0)
- moved R_PW 297.1 mm to (-32.0, -47.0)
- moved U1 157.4 mm to (-174.0, 0.00)
- moved C_UR0 101.6 mm to (-126.0, -70.0)
- moved X1 95.7 mm to (-122.0, -23.0)
- moved C_UR1 51.3 mm to (-99.0, -28.0), turned to 90 degrees
Connections:
- removed net 5V_ARD: J_PZ_EXT.2, LED_RGB.1, LED_RGB.2, LED_RGB.3, R_MIDI_2.2
- removed net 5V_PW: C_VR_1.1, R_PW.2, U_VR_5V.3
- removed net LED_B: R_LED_B.2
- removed net LED_G: R_LED_G.2
- removed net LED_R: R_LED_R.2
- removed net MUX_2: J_PZ_EXT.7
- removed net MUX_A: J_PZ_EXT.6
- removed net MUX_B: J_PZ_EXT.5
- removed net MUX_C: J_PZ_EXT.4
- removed net MUX_D: J_PZ_EXT.3
- removed net N$1: F_PW.2, J_PW.1
- removed net N$9: LED_RGB.6, R_LED_G.1
- removed net RX: R_MIDI_1.2
- removed net TX: R_MIDI_0.2
- removed net USB_5V: C_UR0.1, C_UR1.1, U$1.16, X1.VBUS
- new net 3V3: C_ESP_2.1, C_VR_3.1, MOTPOT_0.3V3, MOTPOT_1.3V3, MOTPOT_2.3V3, R_ESP0.2, R_ESP1.2, R_ESP2.2, R_ESP3.2, R_PW1.2, U1.2, U_VR_1.3
- new net 5V: C_DR_0.1, C_DR_1.1, C_VR_1.1, LED_RGB.1, R_PW.2, U_DR_0.10, U_DR_0.20, U_DR_1.10, U_DR_1.20, U_VR_0.3
- new net EN: R_ESP2.1, U1.3
- new net GPIO15: R_ESP4.1, U1.23
- new net GPIO2: R_ESP1.1, U1.24
- new net LED_RGB: LED_RGB.4, U1.27
- new net MOT_A_0: MOTPOT_0.MOT_A, U_DR_0.2
- new net MOT_A_1: MOTPOT_1.MOT_A, U_DR_0.12
- new net MOT_A_2: MOTPOT_2.MOT_A, U_DR_1.2
- new net MOT_A_3: U_DR_1.12
- new net MOT_B_0: MOTPOT_0.MOT_B, U_DR_0.9
- new net MOT_B_1: MOTPOT_1.MOT_B, U_DR_0.19
- new net MOT_B_2: MOTPOT_2.MOT_B, U_DR_1.9
- new net MOT_B_3: U_DR_1.19
- new net MOT_EN_0: U_DR_0.1
- new net MOT_EN_1: U_DR_0.11
- new net MOT_EN_2: U_DR_1.1
- new net MOT_EN_3: U_DR_1.11
- new net MPOT_0: MOTPOT_0.MPOT
- new net MPOT_1: MOTPOT_1.MPOT
- new net MPOT_2: MOTPOT_2.MPOT
- new net N$14: U_UR0.8, X_UR0.3
- new net N$7: U_UR0.7, X_UR0.1
- new net NRST: C_ESP_3.1, R_ESP3.1
- new net PMOT_A_0: U_DR_0.3
- new net PMOT_A_1: U_DR_0.13
- new net PMOT_A_2: U_DR_1.3
- new net PMOT_A_3: U_DR_1.13
- new net PMOT_B_0: U_DR_0.8
- new net PMOT_B_1: U_DR_0.18
- new net PMOT_B_2: U_DR_1.8
- new net PMOT_B_3: U_DR_1.18
- new net V33: C_VR_2.1, D3.C, U_VR_1.1
- new net V5: C_VR_0.1, D2.C, U_VR_0.1
- net DTR: now also U_UR0.13; no longer U$1.13
- net GND: now also C_DR_0.2, C_DR_1.2, C_ESP_2.2, C_ESP_3.2, C_VR_2.2, C_VR_3.2, LED_PW1.C, LED_RGB.3, MOTPOT_0.GND, MOTPOT_1.GND, MOTPOT_2.GND, R_ESP4.2, U_DR_0.14, U_DR_0.15, U_DR_0.16, U_DR_0.17, U_DR_0.4, U_DR_0.5, U_DR_0.6, U_DR_0.7, U_DR_1.14, U_DR_1.15, U_DR_1.16, U_DR_1.17, U_DR_1.4, U_DR_1.5, U_DR_1.6, U_DR_1.7, U_UR0.1, U_VR_0.4, U_VR_1.2, U_VR_1.4; no longer J_MIDI.1, J_PW.2, J_PW.3, J_PZ_EXT.1, U$1.1, U_VR_5V.2
- net GPIO0: now also R_ESP0.1, U1.25
- net N$10: now also U1.26; no longer LED_RGB.5, R_LED_R.1
- net N$12: now also U_UR0.2; no longer U$1.2
- net N$13: now also U_UR0.3; no longer U$1.3
- net N$15: now also D1.A, X1.VBUS; no longer J_MIDI.2, R_MIDI_2.1
- net N$16: now also U1.29; no longer J_MIDI.3, R_MIDI_1.1
- net N$17: now also U1.14; no longer J_MIDI.4, R_MIDI_0.1
- net N$2: now also U_UR0.15; no longer U$1.15
- net N$8: now also LED_PW1.A, R_PW1.1; no longer LED_RGB.4, R_LED_B.1
- net RTS: now also U_UR0.14; no longer U$1.14
- net USB_D+: now also U_UR0.5; no longer U$1.5
- net USB_D-: now also U_UR0.6; no longer U$1.6
- net VIN: now also C_UR0.1, C_UR1.1, D1.C, D2.A, D3.A, U_UR0.16; no longer C_VR_0.1, F_PW.1, U_VR_5V.1
