File: 02_Elements/MLP_ESPControlBoard_Rev_1/02_HW/MLP_ESPControlBoard_Rev_1.sch (EAGLE design)
At the start: 27 parts, among them Q1 T_UR0, Q2 T_UR0, U1 ESP-WROOM-03, X1 USB-MICROB

Commit message: Schematic Update
Advanced Schematic, not final
Parts:
- removed F_PW: PTCTHERMISTOR1206, SparkFun-PowerIC:PTCTHERMISTOR1206
- removed J_MIDI: 22-05-7048-04, con-molex:22-05-7048-04
- removed J_PW: (no value), con-shiua-chyuan:SCD-014A
- removed J_PZ_EXT: 22-05-7078-07, con-molex:22-05-7078-07
- removed R_LED_B, R_LED_G, R_LED_R: 330, adafruit:R-US_M1206
- removed R_MIDI_0, R_MIDI_1, R_MIDI_2: 220, adafruit:R-US_M1206
- removed U$1: CH340G, ch340g:CH340G
- removed U_VR_5V: 7805T, adafruit:7805T
- added C_DR_0, C_DR_1, C_ESP_2: 100uF, adafruit:C-USC0805K
- added C_ESP_3: 470pF, adafruit:C-USC0805K
- added C_VR_2: 330nF, adafruit:C-USC1206K
- added C_VR_3: 100nF, adafruit:C-USC1206K
- added D1, D2, D3: MBRA140, SparkFun-DiscreteSemi:MBRA140
- added LED_PW1: (no value), adafruit:LEDSMT1206
- added MOTPOT_0, MOTPOT_1, MOTPOT_2: POLOLU_MOT_POT, PololuMotors:POLOLU_MOT_POT
- added R_ESP0, R_ESP1, R_ESP2, R_ESP3, R_ESP4: 12KOhm, adafruit:R-US_M0805
- added R_PW1: 330Ohm, adafruit:R-US_M1206
- added U_DR_0, U_DR_1: L293DD, st-microelectronics:L293DD
- added U_UR0: CH340G, ch340g:CH340G
- added U_VR_0: MC78GENERICDT, _hhn_78xx_79xx_NCV78xx_d2pak_dpak:MC78GENERICDT
- added U_VR_1: UA78M33DCY, linear:UA78M33DCY
- added X_UR0: 12MHz, adafruit:CRYSTALCTS406
- C_UR0, C_UR1: device adafruit:C-USC1812K -> adafruit:C-USC0805K
- C_VR_0: value 18127C103KAT2A -> 330nF; device adafruit:C-USC1812K -> adafruit:C-USC1206K
- C_VR_1: value C1812F104K2RACTU -> 100nF; device adafruit:C-USC1812K -> adafruit:C-USC1206K
- LED_RGB: value RGBLED5050 -> (none); device adafruit:RGBLED5050 -> SparkFun-LED:WS2812B
Connections:
- removed net 5V_ARD: J_PZ_EXT-2.S, LED_RGB.BLUE_A, LED_RGB.GREEN_A, LED_RGB.RED_A, R_MIDI_2.2
- removed net 5V_PW: C_VR_1.1, R_PW.2, U_VR_5V.VO
- removed net LED_B: R_LED_B.2
- removed net LED_G: R_LED_G.2
- removed net LED_R: R_LED_R.2
- removed net MUX_2: J_PZ_EXT-7.S
- removed net MUX_A: J_PZ_EXT-6.S
- removed net MUX_B: J_PZ_EXT-5.S
- removed net MUX_C: J_PZ_EXT-4.S
- removed net MUX_D: J_PZ_EXT-3.S
- removed net N$1: F_PW.2, J_PW.1
- removed net N$9: LED_RGB.GREEN_C, R_LED_G.1
- removed net RX: R_MIDI_1.2
- removed net TX: R_MIDI_0.2
- removed net USB_5V: C_UR0.1, C_UR1.1, U$1.VCC, X1.VBUS
- new net 3V3: C_ESP_2.1, C_VR_3.1, MOTPOT_0.3V3, MOTPOT_1.3V3, MOTPOT_2.3V3, R_ESP0.2, R_ESP1.2, R_ESP2.2, R_ESP3.2, R_PW1.2, U1.3V3, U_VR_1.VO
- new net 5V: C_DR_0.1, C_DR_1.1, C_VR_1.1, LED_RGB.VDD, R_PW.2, U_DR_0.VS, U_DR_0.VSS, U_DR_1.VS, U_DR_1.VSS, U_VR_0.VOUT
- new net EN: R_ESP2.1, U1.EN
- new net GPIO15: R_ESP4.1, U1.IO15
- new net GPIO2: R_ESP1.1, U1.IO2
- new net LED_RGB: LED_RGB.DIN, U1.IO16
- new net MOT_A_0: MOTPOT_0.MOT_A, U_DR_0.IN1
- new net MOT_A_1: MOTPOT_1.MOT_A, U_DR_0.IN3
- new net MOT_A_2: MOTPOT_2.MOT_A, U_DR_1.IN1
- new net MOT_A_3: U_DR_1.IN3
- new net MOT_B_0: MOTPOT_0.MOT_B, U_DR_0.IN2
- new net MOT_B_1: MOTPOT_1.MOT_B, U_DR_0.IN4
- new net MOT_B_2: MOTPOT_2.MOT_B, U_DR_1.IN2
- new net MOT_B_3: U_DR_1.IN4
- new net MOT_EN_0: U_DR_0.EN1
- new net MOT_EN_1: U_DR_0.EN2
- new net MOT_EN_2: U_DR_1.EN1
- new net MOT_EN_3: U_DR_1.EN2
- new net MPOT_0: MOTPOT_0.MPOT
- new net MPOT_1: MOTPOT_1.MPOT
- new net MPOT_2: MOTPOT_2.MPOT
- new net N$14: U_UR0.XO, X_UR0.2
- new net N$7: U_UR0.XI, X_UR0.1
- new net NRST: C_ESP_3.1, R_ESP3.1
- new net PMOT_A_0: U_DR_0.OUT1
- new net PMOT_A_1: U_DR_0.OUT3
- new net PMOT_A_2: U_DR_1.OUT1
- new net PMOT_A_3: U_DR_1.OUT3
- new net PMOT_B_0: U_DR_0.OUT2
- new net PMOT_B_1: U_DR_0.OUT4
- new net PMOT_B_2: U_DR_1.OUT2
- new net PMOT_B_3: U_DR_1.OUT4
- new net V33: C_VR_2.1, D3.C, U_VR_1.VI
- new net V5: C_VR_0.1, D2.C, U_VR_0.VIN
- net DTR: now also U_UR0.DTR; no longer U$1.DTR
- net GND: now also C_DR_0.2, C_DR_1.2, C_ESP_2.2, C_ESP_3.2, C_VR_2.2, C_VR_3.2, LED_PW1.C, LED_RGB.VSS, MOTPOT_0.GND, MOTPOT_1.GND, MOTPOT_2.GND, R_ESP4.2, U_DR_0.GND@1, U_DR_0.GND@2, U_DR_0.GND@3, U_DR_0.GND@4, U_DR_0.GND@5, U_DR_0.GND@6, U_DR_0.GND@7, U_DR_0.GND@8, U_DR_1.GND@1, U_DR_1.GND@2, U_DR_1.GND@3, U_DR_1.GND@4, U_DR_1.GND@5, U_DR_1.GND@6, U_DR_1.GND@7, U_DR_1.GND@8, U_UR0.GND, U_VR_0.GND, U_VR_1.GND, U_VR_1.GND@1; no longer J_MIDI-1.S, J_PW.2, J_PW.3, J_PZ_EXT-1.S, U$1.GND, U_VR_5V.GND
- net GPIO0: now also R_ESP0.1, U1.IO0
- net N$10: now also U1.IO4; no longer LED_RGB.RED_C, R_LED_R.1
- net N$12: now also U_UR0.TX; no longer U$1.TX
- net N$13: now also U_UR0.RX; no longer U$1.RX
- net N$15: now also D1.A, X1.VBUS; no longer J_MIDI-2.S, R_MIDI_2.1
- net N$16: now also U1.IO5; no longer J_MIDI-3.S, R_MIDI_1.1
- net N$17: now also U1.IO12; no longer J_MIDI-4.S, R_MIDI_0.1
- net N$2: now also U_UR0.RS232; no longer U$1.RS232
- net N$8: now also LED_PW1.A, R_PW1.1; no longer LED_RGB.BLUE_C, R_LED_B.1
- net RTS: now also U_UR0.RTS; no longer U$1.RTS
- net USB_D+: now also U_UR0.D+; no longer U$1.D+
- net USB_D-: now also U_UR0.D-; no longer U$1.D-
- net VIN: now also C_UR0.1, C_UR1.1, D1.C, D2.A, D3.A, U_UR0.VCC; no longer C_VR_0.1, F_PW.1, U_VR_5V.VI
Other:
- note added: "H-Bridge Motor Drivers"
- note added: "Note: There is not motor 3 in this scope os the project"
- note added: "Power Input 3V3"
- note added: "Power Input 5V"
- note added: "UART Serial Adapter"
- note removed: "Arduino Leonardo"
- note removed: "Board Main Connectors"
- note removed: "MIDI Jack Connector"
- note removed: "Note: MIDI Jack Connector is just for experimental use."
- note removed: "Note: The Fuse Current must be determined once built"
- note removed: "Power Connector"
- note removed: "Power Input"
- note removed: "RGB LED"
- moved on the sheet: C_UR0, C_UR1, C_VR_0, C_VR_1, LED_PW, Q1, Q2, R_PW, R_UR0, R_UR1, R_UR2, R_UR3
